File: 4_Fabrication/Version_00/C_KiCad/beer-speed/beer-speed.sch (KiCad schematic (older format))
At the start: 10 parts

Commit message: modif kicad
add prog connector
Parts:
- added R?: R, symbol Device:R
Connections:
- net +3V0: now also J?.2 (Pin_2), R?.1; no longer U?.40 (PF6/~RESET)
- net 1E: now also J?.4 (Pin_4)
- net 1F: now also J?.1 (Pin_1)
- net 1G: now also J?.3 (Pin_3)
- net GND: now also J?.6 (Pin_6)
- net RESET: now reaches J?.5 (Pin_5)
- net RESET: now also U?.40 (PF6/~RESET), R?.2
- no-connect marks 2 -> 7
Other:
- note added: "MISO\n"
- note added: "MOSI"
- note added: "SCK"
Changed lines of the file:
@@
 U 1 1 609937E9
 P 6450 2400
-F 0 "C?" H 6565 2446 50  0000 L CNN
-F 1 "C" H 6565 2355 50  0000 L CNN
+F 0 "C?" V 6700 2400 50  0000 L CNN
+F 1 "C" V 6600 2450 50  0000 L CNN
 F 2 "" H 6488 2250 50  0001 C CNN
 F 3 "~" H 6450 2400 50  0001 C CNN
@@
 U 1 1 609940B6
 P 6450 2800
-F 0 "C?" H 6565 2846 50  0000 L CNN
-F 1 "C" H 6565 2755 50  0000 L CNN
+F 0 "C?" V 6700 2750 50  0000 L CNN
+F 1 "C" V 6600 2750 50  0000 L CNN
 F 2 "" H 6488 2650 50  0001 C CNN
 F 3 "~" H 6450 2800 50  0001 C CNN
@@
 U 1 1 6099431E
 P 6700 2600
-F 0 "Y?" H 6700 2868 50  0000 C CNN
-F 1 "Crystal" H 6700 2777 50  0000 C CNN
+F 0 "Y?" V 7050 2600 50  0000 C CNN
+F 1 "Crystal" V 6950 2500 50  0000 C CNN
 F 2 "" H 6700 2600 50  0001 C CNN
 F 3 "~" H 6700 2600 50  0001 C CNN
@@
 Wire Wire Line
 	7700 5050 7700 4950
-$Comp
-L power:+3V0 #PWR?
-U 1 1 60A14D2A
-P 6950 3100
-F 0 "#PWR?" H 6950 2950 50  0001 C CNN
-F 1 "+3V0" H 6965 3273 50  0000 C CNN
-F 2 "" H 6950 3100 50  0001 C CNN
-F 3 "" H 6950 3100 50  0001 C CNN
-	1    6950 3100
-	1    0    0    -1
-$EndComp
-Wire Wire Line
-	6950 3100 6950 3150
-Wire Wire Line
-	6950 3150 7100 3150
 NoConn ~ 7800 2150
 $Comp
@@
 U 1 1 60A21C4E
 P 6700 1400
-F 0 "J?" H 6750 1717 50  0000 C CNN
-F 1 "Conn_02x03_Odd_Even" H 6750 1626 50  0000 C CNN
+F 0 "J?" H 6500 1750 50  0000 C CNN
+F 1 "Conn_02x03_Odd_Even" H 6700 1650 50  0000 C CNN
 F 2 "" H 6700 1400 50  0001 C CNN
 F 3 "~" H 6700 1400 50  0001 C CNN
@@
 	1    0    0    -1
 $EndComp
+$Comp
+L power:+3V0 #PWR?
+U 1 1 609A547B
+P 7250 1250
+F 0 "#PWR?" H 7250 1100 50  0001 C CNN
+F 1 "+3V0" H 7265 1423 50  0000 C CNN
+F 2 "" H 7250 1250 50  0001 C CNN
+F 3 "" H 7250 1250 50  0001 C CNN
+	1    7250 1250
+	1    0    0    -1
+$EndComp
+Wire Wire Line
+	7000 1300 7250 1300
+Wire Wire Line
+	7250 1300 7250 1250
+$Comp
+L power:GND #PWR?
+U 1 1 609A9D7D
+P 7250 1550
+F 0 "#PWR?" H 7250 1300 50  0001 C CNN
+F 1 "GND" H 7255 1377 50  0000 C CNN
+F 2 "" H 7250 1550 50  0001 C CNN
+F 3 "" H 7250 1550 50  0001 C CNN
+	1    7250 1550
+	1    0    0    -1
+$EndComp
+Wire Wire Line
+	7250 1550 7250 1500
+Wire Wire Line
+	7250 1500 7000 1500
+Wire Wire Line
+	6300 1300 6500 1300
+Wire Wire Line
+	7000 1400 7250 1400
+Text GLabel 6000 1500 0    50   Input ~ 0
+RESET
+Wire Wire Line
+	6300 1400 6500 1400
+Text GLabel 7050 3150 0    50   Input ~ 0
+RESET
+Text GLabel 7250 1400 2    50   Output ~ 0
+1E
+Text Notes 7050 1400 0    50   ~ 0
+MOSI
+Text Notes 6350 1300 0    50   ~ 0
+MISO\n
+Text Notes 6350 1400 0    50   ~ 0
+SCK
+Text GLabel 6300 1300 0    50   Output ~ 0
+1F
+Text GLabel 6300 1400 0    50   Output ~ 0
+1G
+$Comp
+L Device:R R?
+U 1 1 609F3A24
+P 6050 1200
+F 0 "R?" H 5900 1250 50  0000 L CNN
+F 1 "R" H 5900 1150 50  0000 L CNN
+F 2 "" V 5980 1200 50  0001 C CNN
+F 3 "~" H 6050 1200 50  0001 C CNN
+	1    6050 1200
+	1    0    0    -1
+$EndComp
+Wire Wire Line
+	6050 1350 6050 1500
+Wire Wire Line
+	6050 1500 6000 1500
+Wire Wire Line
+	6050 1500 6500 1500
+Connection ~ 6050 1500
+$Comp
+L power:+3V0 #PWR?
+U 1 1 60A0755A
+P 6050 1000
+F 0 "#PWR?" H 6050 850 50  0001 C CNN
+F 1 "+3V0" H 6065 1173 50  0000 C CNN
+F 2 "" H 6050 1000 50  0001 C CNN
+F 3 "" H 6050 1000 50  0001 C CNN
+	1    6050 1000
+	1    0    0    -1
+$EndComp
+Wire Wire Line
+	6050 1050 6050 1000
+Wire Wire Line
+	7100 3150 7050 3150
+NoConn ~ 7100 2350
+NoConn ~ 7100 2750
+NoConn ~ 7100 2850
+NoConn ~ 7100 2950
+NoConn ~ 7100 3050
 $EndSCHEMATC

Commit message: modif kicad
small modif
Other:
- note added: "Affichage"
- note added: "Alimentation"
- note added: "Atmega\n"
- note added: "BeerSpeed"
- note added: "Conecteur 2x3 programation spi"
- note added: "LCD 4 digit || 8 . 8 . : 8 . 8"
- note added: "Pile CR 2032 || 3V"
- note added: "Programmation"
- moved on the sheet: BT?, C?, J?, NT?, P?, R?, SW?, U?, Y?
