File: 4_Fabrication/Version_00/C_KiCad/beer-speed/beer-speed.sch (KiCad schematic (older format))
At the start: 11 parts, among them J1 Conn_02x03_Odd_Even, P1 LCD-S401C52TR, SW1 EG1213, SW2 TM1000Q, U1 ATmega4809-A, Y1 Crystal 8MHz

Commit message: modif kicad
modif kicad
modif datasheet
add 3d
add screen footprint
add sensor footprint
Parts:
- BT1: footprint (none) -> Battery:BS-7-ND-20mm
- C1, C2: value 18 pF -> 16 pF
- P1: footprint (none) -> Display:LCD-S401C52TR
- SW2: footprint (none) -> Sensor:TM1000Q
- Y1: footprint (none) -> Crystal:Crystal_SMD_HC49-SD_HandSoldering
Other:
- note added: "Pile CR 2032 (20 mm) || 3V"
- note removed: "Pile CR 2032 || 3V"
Changed lines of the file:
@@
 Comment2 ""
 Comment3 ""
-Comment4 "Robin Forestier"
+Comment4 "Robin Forestier | Maxime Montandon | Kilyan De Blasio"
 $EndDescr
 $Comp
@@
 P 6600 2650
 F 0 "C1" V 6850 2650 50  0000 L CNN
-F 1 "18 pF" V 6750 2550 50  0000 L CNN
+F 1 "16 pF" V 6750 2550 50  0000 L CNN
 F 2 "Capacitor_SMD:C_0805_2012Metric" H 6638 2500 50  0001 C CNN
 F 3 "https://datasheets.avx.com/C0GNP0-Dielectric.pdf" H 6600 2650 50  0001 C CNN
@@
 P 6600 3050
 F 0 "C2" V 6850 3000 50  0000 L CNN
-F 1 "18 pF" V 6750 3000 50  0000 L CNN
+F 1 "16 pF" V 6750 3000 50  0000 L CNN
 F 2 "Capacitor_SMD:C_0805_2012Metric" H 6638 2900 50  0001 C CNN
 F 3 "https://datasheets.avx.com/C0GNP0-Dielectric.pdf" H 6600 3050 50  0001 C CNN
@@
 F 0 "Y1" V 7200 2850 50  0000 C CNN
 F 1 "Crystal 8MHz" V 7100 2750 50  0000 C CNN
-F 2 "" H 6850 2850 50  0001 C CNN
+F 2 "Crystal:Crystal_SMD_HC49-SD_HandSoldering" H 6850 2850 50  0001 C CNN
 F 3 "https://www.ctscorp.com/wp-content/uploads/ATS-ATSSM.pdf" H 6850 2850 50  0001 C CNN
 F 4 "0,27" H 6850 2850 50  0001 C CNN "prix unite"
@@
 F 0 "SW2" H 8950 5085 50  0000 C CNN
 F 1 "TM1000Q" H 8950 4994 50  0000 C CNN
-F 2 "" H 8950 4800 50  0001 C CNN
+F 2 "Sensor:TM1000Q" H 8950 4800 50  0001 C CNN
 F 3 "https://sten-eswitch-13110800-production.s3.amazonaws.com/system/asset/product_line/data_sheet/128/TM1000.pdf" H 8950 4800 50  0001 C CNN
 F 4 "1.16" H 8950 4800 50  0001 C CNN "prix unite"
@@
 F 0 "BT1" H 2418 1746 50  0000 L CNN
 F 1 "Battery_Cell" H 2418 1655 50  0000 L CNN
-F 2 "" V 2300 1710 50  0001 C CNN
+F 2 "Battery:BS-7-ND-20mm" V 2300 1710 50  0001 C CNN
 F 3 "https://www.memoryprotectiondevices.com/datasheets/BS-7-datasheet.pdf" V 2300 1710 50  0001 C CNN
 F 4 "0.6" H 2300 1650 50  0001 C CNN "prix unite"
@@
 F 0 "P1" H 2700 7215 50  0000 C CNN
 F 1 "LCD-S401C52TR" H 2700 7124 50  0000 C CNN
-F 2 "" H 2400 7200 50  0001 C CNN
+F 2 "Display:LCD-S401C52TR" H 2400 7200 50  0001 C CNN
 F 3 "https://www.lumex.com/spec/LCD-S401C52TR.pdf" H 2400 7200 50  0001 C CNN
 F 4 "3,16" H 2700 5950 50  0001 C CNN "prix unite"
@@
 Alimentation
 Text Notes 1850 950  0    50   ~ 0
-Pile CR 2032 || 3V
+Pile CR 2032 (20 mm) || 3V
 Wire Notes Line
 	1650 7300 3750 7300
@@
 Text Notes 5750 1850 0    50   ~ 0
 Atmega\n
-Text Notes 5350 850  0    236  ~ 0
+Text Notes 4500 1100 0    276  ~ 55
 BeerSpeed
 $EndSCHEMATC

Commit message: creat PCB v0
creat PCB
add archive
Parts:
- BT1: symbol Device:Battery_Cell -> archive:Device_Battery_Cell
- C1, C2: symbol Device:C -> archive:Device_C
- J1: symbol Connector_Generic:Conn_02x03_Odd_Even -> archive:Connector_Generic_Conn_02x03_Odd_Even
- NT1: symbol Device:Net-Tie_2 -> archive:Device_Net-Tie_2
- P1: symbol Display_Character:LCD-S401C52TR -> archive:Display_Character_LCD-S401C52TR
- R1: symbol Device:R -> archive:Device_R
- SW1, SW2: symbol Switch:SW_SPDT -> archive:Switch_SW_SPDT
- U1: symbol MCU_Microchip_ATmega:ATmega4809-A -> archive:MCU_Microchip_ATmega_ATmega4809-A
- Y1: symbol Device:Crystal -> archive:Device_Crystal
Changed lines of the file:
@@
 $EndDescr
 $Comp
-L Device:C C1
+L archive:Device_C C1
 U 1 1 609937E9
 P 6600 2650
@@
 $EndComp
 $Comp
-L Device:C C2
+L archive:Device_C C2
 U 1 1 609940B6
 P 6600 3050
@@
 $EndComp
 $Comp
-L Device:Crystal Y1
+L archive:Device_Crystal Y1
 U 1 1 6099431E
 P 6850 2850
@@
 $EndComp
 $Comp
-L Switch:SW_SPDT SW1
+L archive:Switch_SW_SPDT SW1
 U 1 1 609952D2
 P 2900 1400
@@
 $EndComp
 $Comp
-L Switch:SW_SPDT SW2
+L archive:Switch_SW_SPDT SW2
 U 1 1 60995CBA
 P 8950 4800
@@
 $EndComp
 $Comp
-L Device:Battery_Cell BT1
+L archive:Device_Battery_Cell BT1
 U 1 1 60996023
 P 2300 1650
@@
 $EndComp
 $Comp
-L Display_Character:LCD-S401C52TR P1
+L archive:Display_Character_LCD-S401C52TR P1
 U 1 1 609A8933
 P 2700 5950
@@
 $EndComp
 $Comp
-L MCU_Microchip_ATmega:ATmega4809-A U1
+L archive:MCU_Microchip_ATmega_ATmega4809-A U1
 U 1 1 609ABED1
 P 7850 3800
@@
 	2200 5050 2300 5050
 $Comp
-L power:GND #PWR02
+L archive:power_GND #PWR02
 U 1 1 609C102E
 P 2300 1800
@@
 $EndComp
 $Comp
-L power:GND #PWR09
+L archive:power_GND #PWR09
 U 1 1 609C1776
 P 2000 5050
@@
 $EndComp
 $Comp
-L power:+3V0 #PWR01
+L archive:power_+3V0 #PWR01
 U 1 1 609C2EE0
 P 3200 1200
@@
 $EndComp
 $Comp
-L power:+3V0 #PWR08
+L archive:power_+3V0 #PWR08
 U 1 1 609C5C85
 P 9300 4700
@@
 $EndComp
 $Comp
-L Device:Net-Tie_2 NT1
+L archive:Device_Net-Tie_2 NT1
 U 1 1 609C5F35
 P 6350 3250
@@
 	6350 3350 6350 3450
 $Comp
-L power:GND #PWR06
+L archive:power_GND #PWR06
 U 1 1 609C9A74
 P 6350 3450
@@
 	7850 2400 7850 2300
 $Comp
-L power:+3V0 #PWR03
+L archive:power_+3V0 #PWR03
 U 1 1 60A03461
 P 7850 2300
@@
 $EndComp
 $Comp
-L power:GND #PWR010
+L archive:power_GND #PWR010
 U 1 1 60A07167
 P 7850 5300
@@
 NoConn ~ 7950 2400
 $Comp
-L Connector_Generic:Conn_02x03_Odd_Even J1
+L archive:Connector_Generic_Conn_02x03_Odd_Even J1
 U 1 1 60A21C4E
 P 2850 3450
@@
 $EndComp
 $Comp
-L power:+3V0 #PWR05
+L archive:power_+3V0 #PWR05
 U 1 1 609A547B
 P 3400 3300
@@
 	3400 3350 3400 3300
 $Comp
-L power:GND #PWR07
+L archive:power_GND #PWR07
 U 1 1 609A9D7D
 P 3400 3600
@@
 1G
 $Comp
-L Device:R R1
+L archive:Device_R R1
 U 1 1 609F3A24
 P 2200 3250
@@
 Connection ~ 2200 3550
 $Comp
-L power:+3V0 #PWR04
+L archive:power_+3V0 #PWR04
 U 1 1 60A0755A
 P 2200 3050

Commit message: KiCad PCB V0
First version of KiCad PCB
Parts:
- added H1, H2, H3, H4: MountingHole, MountingHole:MountingHole_3.2mm_M3, symbol archive:Mechanical_MountingHole
Other:
- note added: "trou de fixation"
Changed lines of the file:
@@
 Text Notes 4500 1100 0    276  ~ 55
 BeerSpeed
+$Comp
+L archive:Mechanical_MountingHole H1
+U 1 1 609C059A
+P 4700 6150
+F 0 "H1" H 4800 6196 50  0000 L CNN
+F 1 "MountingHole" H 4800 6105 50  0000 L CNN
+F 2 "MountingHole:MountingHole_3.2mm_M3" H 4700 6150 50  0001 C CNN
+F 3 "~" H 4700 6150 50  0001 C CNN
+	1    4700 6150
+	1    0    0    -1
+$EndComp
+$Comp
+L archive:Mechanical_MountingHole H2
+U 1 1 609C1485
+P 5500 6150
+F 0 "H2" H 5600 6196 50  0000 L CNN
+F 1 "MountingHole" H 5600 6105 50  0000 L CNN
+F 2 "MountingHole:MountingHole_3.2mm_M3" H 5500 6150 50  0001 C CNN
+F 3 "~" H 5500 6150 50  0001 C CNN
+	1    5500 6150
+	1    0    0    -1
+$EndComp
+$Comp
+L archive:Mechanical_MountingHole H3
+U 1 1 609C61A5
+P 4700 6500
+F 0 "H3" H 4800 6546 50  0000 L CNN
+F 1 "MountingHole" H 4800 6455 50  0000 L CNN
+F 2 "MountingHole:MountingHole_3.2mm_M3" H 4700 6500 50  0001 C CNN
+F 3 "~" H 4700 6500 50  0001 C CNN
+	1    4700 6500
+	1    0    0    -1
+$EndComp
+$Comp
+L archive:Mechanical_MountingHole H4
+U 1 1 609CAB8D
+P 5500 6500
+F 0 "H4" H 5600 6546 50  0000 L CNN
+F 1 "MountingHole" H 5600 6455 50  0000 L CNN
+F 2 "MountingHole:MountingHole_3.2mm_M3" H 5500 6500 50  0001 C CNN
+F 3 "~" H 5500 6500 50  0001 C CNN
+	1    5500 6500
+	1    0    0    -1
+$EndComp
+Wire Notes Line
+	4550 6700 6200 6700
+Wire Notes Line
+	6200 6700 6200 5950
+Wire Notes Line
+	6200 5950 4550 5950
+Wire Notes Line
+	4550 5950 4550 6700
+Text Notes 4550 5900 0    50   ~ 0
+trou de fixation
 $EndSCHEMATC
